File: snescart.kicad_pcb (KiCad board)
At the start: 2 copper layers, 101.6 x 38.1 mm, 6 parts, among them P1 CASSETTE, U1 27C512

Commit message: tracks
Parts:
- removed U1: 27C512, Package_DIP:DIP-28_W15.24mm
- added U3: 27C080, Package_DIP:DIP-32_W15.24mm, F.Cu at (186.7, 119.4)
- C3: footprint Capacitor_THT:C_Disc_D4.3mm_W1.9mm_P5.00mm -> Capacitor_THT:CP_Axial_L10.0mm_D4.5mm_P15.00mm_Horizontal
Connections:
- P1 pad 36: (no net) -> GND
- P1 pad 37: (no net) -> Net-(P1-A12)
- P1 pad 38: (no net) -> Net-(P1-A13)
- P1 pad 39: (no net) -> Net-(P1-A14)
- P1 pad 40: (no net) -> Net-(P1-A15)
- P1 pad 41: (no net) -> Net-(P1-A16)
- P1 pad 42: (no net) -> Net-(P1-A17)
- P1 pad 43: (no net) -> Net-(P1-A18)
- P1 pad 44: (no net) -> Net-(P1-A19)
- P1 pad 45: (no net) -> unconnected-(P1-A20-Pad45)
- P1 pad 46: (no net) -> unconnected-(P1-A21-Pad46)
- P1 pad 47: (no net) -> unconnected-(P1-A22-Pad47)
- P1 pad 48: (no net) -> unconnected-(P1-A23-Pad48)
- P1 pad 49: (no net) -> unconnected-(P1-ROMSEL-Pad49)
- P1 pad 50: (no net) -> Net-(P1-D4)
- P1 pad 51: (no net) -> Net-(P1-D5)
- P1 pad 54: (no net) -> unconnected-(P1-WR-Pad54)
- P1 pad 55: (no net) -> Net-(P1-CIC1)
- P1 pad 56: (no net) -> Net-(P1-CIC3)
- P1 pad 57: (no net) -> unconnected-(P1-SYSCK-Pad57)
- P1 pad 58: (no net) -> VCC
- P1 pad 59: (no net) -> unconnected-(P1-PA1-Pad59)
- P1 pad 60: (no net) -> unconnected-(P1-PA3-Pad60)
Routing:
- net GND: track 0.00 -> 39.8 mm, vias 0 -> 5
- net Net-(P1-A12): track 0.00 -> 25.1 mm, vias 0 -> 1

Commit message: abababa
Routing:
- net VCC: track 0.00 -> 6.79 mm
Changed lines of the file:
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@@
   (net 52 "unconnected-(P1-WR-Pad54)")
   (net 53 "unconnected-(P1-SYSCK-Pad57)")
-  (net 54 "unconnected-(P1-PA1-Pad59)")
-  (net 55 "unconnected-(P1-PA3-Pad60)")
-  (net 56 "Net-(P1-D6)")
-  (net 57 "Net-(P1-D7)")
-  (net 58 "unconnected-(U3-~{CE}-Pad22)")
-  (net 59 "unconnected-(U3-~{OE}-Pad24)")
+  (net 54 "Net-(P1-D6)")
+  (net 55 "Net-(P1-D7)")
+  (net 56 "unconnected-(U3-~{CE}-Pad22)")
+  (net 57 "unconnected-(U3-~{OE}-Pad24)")
   (footprint "Capacitor_THT:C_Disc_D4.3mm_W1.9mm_P5.00mm" (layer "F.Cu")
     (at 171.45 115.57)
@@
       (net 51 "Net-(P1-D5)") (pinfunction "D5") (pintype "tri_state"))
     (pad "20" thru_hole oval (at 15.24 30.48 270) (size 1.6 1.6) (drill 0.8) (layers "*.Cu" "*.Mask")
-      (net 56 "Net-(P1-D6)") (pinfunction "D6") (pintype "tri_state"))
+      (net 54 "Net-(P1-D6)") (pinfunction "D6") (pintype "tri_state"))
     (pad "21" thru_hole oval (at 15.24 27.94 270) (size 1.6 1.6) (drill 0.8) (layers "*.Cu" "*.Mask")
-      (net 57 "Net-(P1-D7)") (pinfunction "D7") (pintype "tri_state"))
+      (net 55 "Net-(P1-D7)") (pinfunction "D7") (pintype "tri_state"))
     (pad "22" thru_hole oval (at 15.24 25.4 270) (size 1.6 1.6) (drill 0.8) (layers "*.Cu" "*.Mask")
-      (net 58 "unconnected-(U3-~{CE}-Pad22)") (pinfunction "~{CE}") (pintype "input"))
+      (net 56 "unconnected-(U3-~{CE}-Pad22)") (pinfunction "~{CE}") (pintype "input"))
     (pad "23" thru_hole oval (at 15.24 22.86 270) (size 1.6 1.6) (drill 0.8) (layers "*.Cu" "*.Mask")
       (net 4 "Net-(P1-A10)") (pinfunction "A10") (pintype "input"))
     (pad "24" thru_hole oval (at 15.24 20.32 270) (size 1.6 1.6) (drill 0.8) (layers "*.Cu" "*.Mask")
-      (net 59 "unconnected-(U3-~{OE}-Pad24)") (pinfunction "~{OE}") (pintype "input"))
+      (net 57 "unconnected-(U3-~{OE}-Pad24)") (pinfunction "~{OE}") (pintype "input"))
     (pad "25" thru_hole oval (at 15.24 17.78 270) (size 1.6 1.6) (drill 0.8) (layers "*.Cu" "*.Mask")
       (net 3 "Net-(P1-A11)") (pinfunction "A11") (pintype "input"))
@@
     (pad "51" smd rect (at -10 2.952) (size 1.27 5.588) (layers "F.Cu" "B.Paste" "B.Mask")
       (net 51 "Net-(P1-D5)") (pinfunction "D5") (pintype "bidirectional"))
-    (pad "54" smd rect (at -12.5 3) (size 1.27 5.588) (layers "F.Cu" "B.Paste" "B.Mask")
+    (pad "52" smd rect (at -12.5 3) (size 1.27 5.588) (layers "F.Cu" "B.Paste" "B.Mask"))
+    (pad "53" smd rect (at -15 3) (size 1.27 5.588) (layers "F.Cu" "B.Paste" "B.Mask"))
+    (pad "54" smd rect (at -17.5 2.952) (size 1.27 5.588) (layers "F.Cu" "B.Paste" "B.Mask")
       (net 52 "unconnected-(P1-WR-Pad54)") (pinfunction "WR") (pintype "unspecified"))
-    (pad "55" smd rect (at -15 3) (size 1.27 5.588) (layers "F.Cu" "B.Paste" "B.Mask")
+    (pad "55" smd rect (at -20 3) (size 1.27 5.588) (layers "F.Cu" "B.Paste" "B.Mask")
       (net 27 "Net-(P1-CIC1)") (pinfunction "CIC1") (pintype "unspecified"))
-    (pad "56" smd rect (at -17.5 2.952) (size 1.27 5.588) (layers "F.Cu" "B.Paste" "B.Mask")
+    (pad "56" smd rect (at -22.5 3) (size 1.27 5.588) (layers "F.Cu" "B.Paste" "B.Mask")
       (net 24 "Net-(P1-CIC3)") (pinfunction "CIC3") (pintype "unspecified"))
-    (pad "57" smd rect (at -20 3) (size 1.27 5.588) (layers "F.Cu" "B.Paste" "B.Mask")
+    (pad "57" smd rect (at -25 3) (size 1.27 5.588) (layers "F.Cu" "B.Paste" "B.Mask")
       (net 53 "unconnected-(P1-SYSCK-Pad57)") (pinfunction "SYSCK") (pintype "unspecified"))
-    (pad "58" smd rect (at -22.5 3) (size 1.27 5.588) (layers "F.Cu" "B.Paste" "B.Mask")
+    (pad "58" smd rect (at -27.94 3) (size 1.778 5.588) (layers "F.Cu" "B.Paste" "B.Mask")
       (net 2 "VCC") (pinfunction "+5V") (pintype "power_in"))
-    (pad "59" smd rect (at -25 3) (size 1.27 5.588) (layers "F.Cu" "B.Paste" "B.Mask")
-      (net 54 "unconnected-(P1-PA1-Pad59)") (pinfunction "PA1") (pintype "unspecified"))
-    (pad "60" smd rect (at -27.94 3) (size 1.778 5.588) (layers "F.Cu" "B.Paste" "B.Mask")
-      (net 55 "unconnected-(P1-PA3-Pad60)") (pinfunction "PA3") (pintype "unspecified"))
   )
   (footprint "Capacitor_THT:C_Disc_D4.3mm_W1.9mm_P5.00mm" (layer "F.Cu")
@@
   (via (at 178.435 137.795) (size 0.8) (drill 0.4) (layers "F.Cu" "B.Cu") (net 1))
   (via (at 187.325 137.795) (size 0.8) (drill 0.4) (layers "F.Cu" "B.Cu") (net 1))
+  (segment (start 117.035 146.685) (end 117.035 139.895) (width 1.27) (layer "F.Cu") (net 2))
   (segment (start 169.975 140.2098) (end 170.7388 139.446) (width 0.254) (layer "F.Cu") (net 37))
   (segment (start 175.117 129.2446) (end 173.4312 127.5588) (width 0.254) (layer "F.Cu") (net 37))

Commit message: track
Parts:
- moved C3 5.30 mm to (132.1, 119.2)
- moved U3 2.54 mm to (184.2, 119.4)
Routing:
- net GND: track 39.8 -> 27.9 mm
Changed lines of the file:
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@@
       (layer "B.Paste" (type "Bottom Solder Paste"))
       (layer "B.SilkS" (type "Bottom Silk Screen"))
-      (copper_finish "None")
+      (copper_finish "ENIG")
       (dielectric_constraints no)
+      (edge_connector yes)
     )
     (pad_to_mask_clearance 0)
@@
   )
   (footprint "Package_DIP:DIP-32_W15.24mm" (layer "F.Cu")
-    (at 186.69 119.375 -90)
+    (at 184.15 119.375 -90)
     (descr "32-lead though-hole mounted DIP package, row spacing 15.24 mm (600 mils)")
     (tags "THT DIP DIL PDIP 2.54mm 15.24mm 600mil")
@@
   )
   (footprint "Capacitor_THT:CP_Axial_L10.0mm_D4.5mm_P15.00mm_Horizontal" (layer "F.Cu")
-    (at 132.08 124.54 -90)
+    (at 132.08 119.239 -90)
     (descr "CP, Axial series, Axial, Horizontal, pin pitch=15mm, , length*diameter=10*4.5mm^2, Electrolytic Capacitor, , http://www.vishay.com/docs/28325/021asm.pdf")
     (tags "CP Axial series Axial Horizontal pin pitch 15mm  length 10mm diameter 4.5mm Electrolytic Capacitor")
@@
     (property "ki_keywords" "cap capacitor")
     (attr through_hole)
-    (fp_text reference "C3" (at 7.5 -3.37 -90) (layer "F.SilkS")
+    (fp_text reference "C3" (at 12.206 -3.429 -90) (layer "F.SilkS")
         (effects (font (size 1 1) (thickness 0.15)))
     )
@@
     (effects (font (size 1.5 1.5) (thickness 0.3) bold) (justify left bottom))
   )
-  (segment (start 173.99 137.795) (end 176.53 137.795) (width 1.905) (layer "F.Cu") (net 1))
   (segment (start 180.34 137.795) (end 187.325 137.795) (width 1.905) (layer "F.Cu") (net 1))
   (segment (start 176.53 137.795) (end 178.435 137.795) (width 1.905) (layer "F.Cu") (net 1))
   (segment (start 178.435 137.795) (end 180.34 137.795) (width 1.905) (layer "F.Cu") (net 1))
-  (segment (start 172.975 138.81) (end 173.99 137.795) (width 1.905) (layer "F.Cu") (net 1))
   (segment (start 189.23 137.795) (end 193.04 137.795) (width 1.905) (layer "F.Cu") (net 1))
   (segment (start 193.04 137.795) (end 193.04 126.365) (width 1.905) (layer "F.Cu") (net 1))
-  (segment (start 172.975 146.733) (end 172.975 138.81) (width 1.905) (layer "F.Cu") (net 1))
   (segment (start 187.325 137.795) (end 189.23 137.795) (width 1.905) (layer "F.Cu") (net 1))
-  (via (at 189.23 137.795) (size 0.8) (drill 0.4) (layers "F.Cu" "B.Cu") (net 1))
-  (via (at 180.34 137.795) (size 0.8) (drill 0.4) (layers "F.Cu" "B.Cu") (net 1))
-  (via (at 176.53 137.795) (size 0.8) (drill 0.4) (layers "F.Cu" "B.Cu") (net 1))
-  (via (at 178.435 137.795) (size 0.8) (drill 0.4) (layers "F.Cu" "B.Cu") (net 1))
-  (via (at 187.325 137.795) (size 0.8) (drill 0.4) (layers "F.Cu" "B.Cu") (net 1))
+  (via (at 189.357 137.414) (size 0.8) (drill 0.4) (layers "F.Cu" "B.Cu") (net 1))
+  (via (at 181.102 137.541) (size 0.8) (drill 0.4) (layers "F.Cu" "B.Cu") (net 1))
+  (via (at 176.276 137.541) (size 0.8) (drill 0.4) (layers "F.Cu" "B.Cu") (net 1))
+  (via (at 178.816 137.541) (size 0.8) (drill 0.4) (layers "F.Cu" "B.Cu") (net 1))
+  (via (at 186.944 137.414) (size 0.8) (drill 0.4) (layers "F.Cu" "B.Cu") (net 1))
   (segment (start 117.035 146.685) (end 117.035 139.895) (width 1.27) (layer "F.Cu") (net 2))
-  (segment (start 169.975 140.2098) (end 170.7388 139.446) (width 0.254) (layer "F.Cu") (net 37))
-  (segment (start 175.117 129.2446) (end 173.4312 127.5588) (width 0.254) (layer "F.Cu") (net 37))
-  (segment (start 171.2976 138.8872) (end 171.2976 136.6012) (width 0.254) (layer "F.Cu") (net 37))
-  (segment (start 175.1076 135.8392) (end 175.117 135.8298) (width 0.254) (layer "F.Cu") (net 37))
-  (segment (start 170.7388 139.446) (end 171.2976 138.8872) (width 0.254) (layer "F.Cu") (net 37))
+  (segment (start 175.133 135.8458) (end 175.117 135.8298) (width 0.254) (layer "F.Cu") (net 37))
   (segment (start 169.975 146.685) (end 169.975 140.2098) (width 0.254) (layer "F.Cu") (net 37))
   (segment (start 173.4312 126.2888) (end 173.3804 126.238) (width 0.254) (layer "F.Cu") (net 37))
-  (segment (start 171.2976 136.6012) (end 174.3456 136.6012) (width 0.254) (layer "F.Cu") (net 37))
-  (segment (start 174.3456 136.6012) (end 175.1076 135.8392) (width 0.254) (layer "F.Cu") (net 37))
   (segment (start 173.4312 127.5588) (end 173.4312 126.2888) (width 0.254) (layer "F.Cu") (net 37))
+  (segment (start 174.752 137.541) (end 175.133 137.16) (width 0.254) (layer "F.Cu") (net 37))
+  (segment (start 175.133 137.16) (end 175.133 135.8458) (width 0.254) (layer "F.Cu") (net 37))
+  (segment (start 171.2976 137.5664) (end 171.323 137.541) (width 0.254) (layer "F.Cu") (net 37))
+  (segment (start 169.975 140.2098) (end 171.2976 138.8872) (width 0.254) (layer "F.Cu") (net 37))
   (segment (start 175.117 135.8298) (end 175.117 129.2446) (width 0.254) (layer "F.Cu") (net 37))
+  (segment (start 171.2976 138.8872) (end 171.2976 137.5664) (width 0.254) (layer "F.Cu") (net 37))
+  (segment (start 175.117 129.2446) (end 173.4312 127.5588) (width 0.254) (layer "F.Cu") (net 37))
+  (segment (start 171.323 137.541) (end 174.752 137.541) (width 0.254) (layer "F.Cu") (net 37))
   (via (at 173.3804 126.238) (size 0.8) (drill 0.4) (layers "F.Cu" "B.Cu") (net 37))
   (zone (net 1) (net_name "GND") (layer "F.Cu") (hatch edge 0.5)

Commit message: funny cap
Parts:
- C1: footprint Capacitor_THT:C_Disc_D4.3mm_W1.9mm_P5.00mm -> Library:CapacitorSpecial
- C2: footprint Capacitor_THT:C_Disc_D4.3mm_W1.9mm_P5.00mm -> Library:Capacitor
- C3: footprint Capacitor_THT:CP_Axial_L10.0mm_D4.5mm_P15.00mm_Horizontal -> Library:Capacitor
- moved C3 6.36 mm to (132.1, 125.6)
Connections:
- P1 pad 52: (no net) -> Net-(P1-D6)
- P1 pad 53: (no net) -> Net-(P1-D7)
Routing:
- net GND: track 27.9 -> 35.9 mm
- net Net-(P1-A12): track 25.3 -> 22.5 mm

Commit message: date
Parts:
- added REF**: Logo, Library:Logo, F.Cu at (138.7, 116.6)
- renumbered U3 to U1
Other:
- outline, holes or cut-outs redrawn
- board text added: "1990"
Changed lines of the file:
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@@
   (net 54 "Net-(P1-D6)")
   (net 55 "Net-(P1-D7)")
-  (net 56 "unconnected-(U3-~{CE}-Pad22)")
-  (net 57 "unconnected-(U3-~{OE}-Pad24)")
+  (net 56 "unconnected-(U1-~{CE}-Pad22)")
+  (net 57 "unconnected-(U1-~{OE}-Pad24)")
   (footprint "Library:Capacitor" (layer "F.Cu")
     (at 171.45 115.57)
@@
         (effects (font (size 1 1) (thickness 0.15)))
     )
-    (fp_text user "${REFERENCE}" (at 0 2.5 unlocked) (layer "F.Fab")
+    (fp_text user "${REFERENCE}" (at -9.398 0.254 unlocked) (layer "F.Fab")
         (effects (font (size 1 1) (thickness 0.15)))
     )
@@
     (pad "2" thru_hole circle (at 6.35 0) (size 2.286 2.286) (drill 1) (layers "*.Cu" "*.Mask")
       (net 1 "GND") (pintype "passive"))
+  )
+  (footprint "Library:Logo" (layer "F.Cu")
+    (at 138.684 116.586)
+    (attr smd)
+    (fp_text reference "REF**" (at 0 -0.5 unlocked) (layer "F.SilkS") hide
+        (effects (font (size 1 1) (thickness 0.1)))
+    )
+    (fp_text value "Logo" (at 0 1 unlocked) (layer "F.Fab") hide
+        (effects (font (size 1 1) (thickness 0.15)))
+    )
+    (fp_line (start -1.25 -1.25) (end -0.5 -0.5)
+      (stroke (width 0.1) (type default)) (layer "F.SilkS"))
+    (fp_line (start -0.5 -0.5) (end -0.5 1.25)
+      (stroke (width 0.1) (type default)) (layer "F.SilkS"))
+    (fp_line (start -0.5 -0.5) (end 0.25 -1.25)
+      (stroke (width 0.1) (type default)) (layer "F.SilkS"))
+    (fp_line (start 0 -0.75) (end 0 1.25)
+      (stroke (width 0.1) (type default)) (layer "F.SilkS"))
+    (fp_line (start 0 1.25) (end 0.25 1.5)
+      (stroke (width 0.1) (type default)) (layer "F.SilkS"))
+    (fp_line (start 0.25 1.5) (end 1 1.5)
+      (stroke (width 0.1) (type default)) (layer "F.SilkS"))
+    (fp_line (start 0.5 -1.25) (end 0 -0.75)
+      (stroke (width 0.1) (type default)) (layer "F.SilkS"))
+    (fp_line (start 1 1.5) (end 1.5 1)
+      (stroke (width 0.1) (type default)) (layer "F.SilkS"))
+    (fp_line (start 1.25 -1.25) (end 0.5 -1.25)
+      (stroke (width 0.1) (type default)) (layer "F.SilkS"))
+    (fp_line (start 1.5 -1) (end 1.25 -1.25)
+      (stroke (width 0.1) (type default)) (layer "F.SilkS"))
+    (fp_line (start 1.5 -0.5) (end 1.5 -1)
+      (stroke (width 0.1) (type default)) (layer "F.SilkS"))
+    (fp_line (start 1.5 0.25) (end 1 0.25)
+      (stroke (width 0.1) (type default)) (layer "F.SilkS"))
+    (fp_line (start 1.5 1) (end 1.5 0.25)
+      (stroke (width 0.1) (type default)) (layer "F.SilkS"))
+    (fp_circle (center 0 0) (end 0 -2)
+      (stroke (width 0.1) (type default)) (fill none) (layer "F.SilkS"))
   )
   (footprint "Package_DIP:DIP-32_W15.24mm" (layer "F.Cu")
@@
     (property "ki_keywords" "OTP EPROM 8MiBit")
     (attr through_hole)
-    (fp_text reference "U3" (at 7.62 -2.33 90) (layer "F.SilkS")
+    (fp_text reference "U1" (at -2.154 -0.254 -180) (layer "F.SilkS")
         (effects (font (size 1 1) (thickness 0.15)))
     )
@@
       (net 55 "Net-(P1-D7)") (pinfunction "D7") (pintype "tri_state"))
     (pad "22" thru_hole oval (at 15.24 25.4 270) (size 1.6 1.6) (drill 0.8) (layers "*.Cu" "*.Mask")
-      (net 56 "unconnected-(U3-~{CE}-Pad22)") (pinfunction "~{CE}") (pintype "input"))
+      (net 56 "unconnected-(U1-~{CE}-Pad22)") (pinfunction "~{CE}") (pintype "input"))
     (pad "23" thru_hole oval (at 15.24 22.86 270) (size 1.6 1.6) (drill 0.8) (layers "*.Cu" "*.Mask")
       (net 4 "Net-(P1-A10)") (pinfunction "A10") (pintype "input"))
     (pad "24" thru_hole oval (at 15.24 20.32 270) (size 1.6 1.6) (drill 0.8) (layers "*.Cu" "*.Mask")
-      (net 57 "unconnected-(U3-~{OE}-Pad24)") (pinfunction "~{OE}") (pintype "input"))
+      (net 57 "unconnected-(U1-~{OE}-Pad24)") (pinfunction "~{OE}") (pintype "input"))
     (pad "25" thru_hole oval (at 15.24 17.78 270) (size 1.6 1.6) (drill 0.8) (layers "*.Cu" "*.Mask")
       (net 3 "Net-(P1-A11)") (pinfunction "A11") (pintype "input"))
@@
   (gr_line (start 97.79 123.19) (end 93.98 123.19)
     (stroke (width 0.1) (type default)) (layer "Edge.Cuts"))
-  (gr_circle (center 100.33 116.205) (end 99.695 116.205)
+  (gr_circle (center 100.33 116.84) (end 99.568 116.713)
     (stroke (width 0.1) (type default)) (fill none) (layer "Edge.Cuts"))
   (gr_line (start 115.57 151.13) (end 115.57 149.225)
@@
   (gr_line (start 191.77 116.84) (end 191.77 113.03)
     (stroke (width 0.1) (type default)) (layer "Edge.Cuts"))
-  (gr_text "SHVC-1AON-20" (at 99.06 115.57) (layer "F.SilkS")
+  (gr_text "SHVC-1AON-20" (at 98.933 115.697) (layer "F.SilkS")
+    (effects (font (size 1.5 1.5) (thickness 0.3) bold) (justify left bottom))
+  )
+  (gr_text "1990" (at 98.679 135.255 90) (layer "F.SilkS")
     (effects (font (size 1.5 1.5) (thickness 0.3) bold) (justify left bottom))
   )
@@
     (polygon
       (pts
+        (xy 94.615 134.493)
+        (xy 96.012 133.096)
+        (xy 95.758 125.222)
+        (xy 97.79 125.222)
+        (xy 98.679 123.825)
+        (xy 97.663 122.809)
+        (xy 95.25 122.809)
+        (xy 94.615 121.793)
         (xy 94.615 113.665)
         (xy 194.945 113.665)
-        (xy 194.945 142.875)
-        (xy 94.615 142.875)
+        (xy 194.945 138.684)
+        (xy 94.615 139.065)
       )
     )

Commit message: jkfjf
Parts:
- moved C1 1.24 mm to (110.4, 133.3)
Routing:
- net VCC: track 6.79 -> 14.9 mm, vias 0 -> 3
Other:
- outline, holes or cut-outs redrawn
Changed lines of the file:
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@@
     (fp_line (start 1.5 1) (end 1.5 0.25)
       (stroke (width 0.1) (type default)) (layer "F.SilkS"))
-    (fp_circle (center 0 0) (end 0 -2)
+    (fp_circle (center 0 0) (end 0 -1.905)
       (stroke (width 0.1) (type default)) (fill none) (layer "F.SilkS"))
   )
@@
         (effects (font (size 1 1) (thickness 0.15)))
     )
-    (fp_line (start -4.445 0) (end -0.635 0)
+    (fp_line (start -3.175 0) (end -0.635 0)
       (stroke (width 0.1) (type default)) (layer "F.SilkS"))
     (fp_line (start -0.635 -1.27) (end -0.635 1.27)
@@
     (fp_line (start 0.635 -1.27) (end 0.635 1.27)
       (stroke (width 0.1) (type default)) (layer "F.SilkS"))
-    (fp_line (start 0.635 0) (end 4.445 0)
-      (stroke (width 0.1) (type default)) (layer "F.SilkS"))
-    (pad "1" thru_hole rect (at -6.35 0 270) (size 2.286 2.286) (drill 1) (layers "*.Cu" "*.Mask")
+    (fp_line (start 0.635 0) (end 2.54 0)
+      (stroke (width 0.1) (type default)) (layer "F.SilkS"))
+    (pad "1" thru_hole rect (at -5.715 0 270) (size 2.286 2.286) (drill 1) (layers "*.Cu" "*.Mask")
       (net 25 "unconnected-(C3-Pad1)") (pintype "passive") (thermal_bridge_angle 45))
-    (pad "2" thru_hole circle (at 6.35 0 270) (size 2.286 2.286) (drill 1) (layers "*.Cu" "*.Mask")
+    (pad "2" thru_hole circle (at 5.08 0 270) (size 2.286 2.286) (drill 1) (layers "*.Cu" "*.Mask")
       (net 26 "unconnected-(C3-Pad2)") (pintype "passive"))
   )
@@
   )
   (footprint "Library:CapacitorSpecial" (layer "F.Cu")
-    (at 110.49 134.58 90)
+    (at 110.363 133.35 90)
     (property "Sheetfile" "snescart.kicad_sch")
     (property "Sheetname" "")
@@
         (effects (font (size 1 1) (thickness 0.15)))
     )
-    (fp_line (start -3.175 -3.175) (end 3.175 -3.175)
-      (stroke (width 0.1) (type default)) (layer "F.SilkS"))
-    (fp_line (start -3.175 -1.27) (end -3.175 -3.175)
-      (stroke (width 0.1) (type default)) (layer "F.SilkS"))
-    (fp_line (start 3.175 -3.175) (end 3.175 -1.27)
-      (stroke (width 0.1) (type default)) (layer "F.SilkS"))
-    (pad "1" thru_hole circle (at -3.175 0 90) (size 1.524 1.524) (drill 0.762) (layers "*.Cu" "*.Mask")
+    (fp_line (start -1.905 -3.175) (end 1.905 -3.175)
+      (stroke (width 0.1) (type default)) (layer "F.SilkS"))
+    (fp_line (start -1.905 -1.27) (end -1.905 -3.175)
+      (stroke (width 0.1) (type default)) (layer "F.SilkS"))
+    (fp_line (start -1.27 -3.81) (end -1.27 -2.54)
+      (stroke (width 0.1) (type default)) (layer "F.SilkS"))
+    (fp_line (start 1.27 -3.81) (end 1.27 -2.54)
+      (stroke (width 0.1) (type default)) (layer "F.SilkS"))
+    (fp_line (start 1.905 -4.445) (end 3.175 -4.445)
+      (stroke (width 0.1) (type default)) (layer "F.SilkS"))
+    (fp_line (start 1.905 -3.175) (end 1.905 -1.27)
+      (stroke (width 0.1) (type default)) (layer "F.SilkS"))
+    (fp_line (start 2.54 -3.81) (end 2.54 -5.08)
+      (stroke (width 0.1) (type default)) (layer "F.SilkS"))
+    (pad "1" thru_hole circle (at -1.905 0 90) (size 1.524 1.524) (drill 0.762) (layers "*.Cu" "*.Mask")
       (net 1 "GND") (pintype "passive"))
-    (pad "2" thru_hole circle (at 3.175 0 90) (size 1.524 1.524) (drill 0.762) (layers "*.Cu" "*.Mask")
+    (pad "2" thru_hole circle (at 1.905 0 90) (size 1.524 1.524) (drill 0.762) (layers "*.Cu" "*.Mask")
       (net 2 "VCC") (pintype "passive"))
   )
@@
   (gr_line (start 97.79 123.19) (end 93.98 123.19)
     (stroke (width 0.1) (type default)) (layer "Edge.Cuts"))
-  (gr_circle (center 100.33 116.84) (end 99.568 116.713)
+  (gr_circle (center 100.33 117.84549) (end 99.187 117.856)
     (stroke (width 0.1) (type default)) (fill none) (layer "Edge.Cuts"))
   (gr_line (start 115.57 151.13) (end 115.57 149.225)
@@
   (gr_line (start 191.77 116.84) (end 191.77 113.03)
     (stroke (width 0.1) (type default)) (layer "Edge.Cuts"))
-  (gr_text "SHVC-1AON-20" (at 98.933 115.697) (layer "F.SilkS")
+  (gr_text "SHVC-1AON-20" (at 98.933 115.824) (layer "F.SilkS")
     (effects (font (size 1.5 1.5) (thickness 0.3) bold) (justify left bottom))
   )
@@
   (via (at 179.07 137.287) (size 0.8) (drill 0.4) (layers "F.Cu" "B.Cu") (net 1))
   (via (at 186.817 137.287) (size 0.8) (drill 0.4) (layers "F.Cu" "B.Cu") (net 1))
+  (segment (start 117.856 136.906) (end 117.856 134.62) (width 1.905) (layer "F.Cu") (net 2))
   (segment (start 117.035 146.685) (end 117.035 139.895) (width 1.905) (layer "F.Cu") (net 2))
+  (segment (start 117.856 134.62) (end 117.856 132.207) (width 1.905) (layer "F.Cu") (net 2))
+  (segment (start 117.856 132.207) (end 117.856 132.08) (width 1.905) (layer "F.Cu") (net 2))
+  (segment (start 117.035 139.895) (end 117.035 137.727) (width 1.905) (layer "F.Cu") (net 2))
+  (segment (start 117.035 137.727) (end 117.856 136.906) (width 1.905) (layer "F.Cu") (net 2))
+  (via (at 117.856 136.906) (size 0.8) (drill 0.4) (layers "F.Cu" "B.Cu") (net 2))
+  (via (at 117.856 134.62) (size 0.8) (drill 0.4) (layers "F.Cu" "B.Cu") (net 2))
+  (via (at 117.856 132.207) (size 0.8) (drill 0.4) (layers "F.Cu" "B.Cu") (net 2))
   (segment (start 174.432991 135.763) (end 173.101 135.763) (width 0.25) (layer "F.Cu") (net 37))
   (segment (start 169.975 146.685) (end 169.975 140.2098) (width 0.254) (layer "F.Cu") (net 37))
@@
     (polygon
       (pts
-        (xy 94.615 134.493)
-        (xy 96.012 133.096)
+        (xy 94.615 133.35)
+        (xy 95.758 131.826)
         (xy 95.758 125.222)
         (xy 97.79 125.222)

Commit message: asdjus
Parts:
- moved C2 4.16 mm to (175.5, 116.5)
Routing:
- net VCC: track 14.9 -> 46.8 mm
Other:
- outline, holes or cut-outs redrawn
- board text added: "MASK ROM"
