File: snescart.kicad_pcb (KiCad board)
At the start: 2 copper layers, 101.6 x 38.1 mm, 7 parts, among them P1 CASSETTE, U1 27C080

Commit message: edfhgdfhg
Parts:
- moved C2 1.65 mm to (177.2, 116.5)
- moved C1 0.51 mm to (110.4, 132.8)
Routing:
- net VCC: track 46.8 -> 63.0 mm, vias 3 -> 6
- net GND: track 35.9 -> 38.6 mm
Other:
- outline, holes or cut-outs redrawn
Changed lines of the file:
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@@
   (net 57 "unconnected-(U1-~{OE}-Pad24)")
   (footprint "Library:Capacitor" (layer "F.Cu")
-    (at 175.514 116.459)
+    (at 177.165 116.459)
     (property "Sheetfile" "snescart.kicad_sch")
     (property "Sheetname" "")
@@
         (effects (font (size 1 1) (thickness 0.15)))
     )
-    (fp_line (start -1.25 -1.25) (end -0.5 -0.5)
-      (stroke (width 0.1) (type default)) (layer "F.SilkS"))
-    (fp_line (start -0.5 -0.5) (end -0.5 1.25)
-      (stroke (width 0.1) (type default)) (layer "F.SilkS"))
-    (fp_line (start -0.5 -0.5) (end 0.25 -1.25)
-      (stroke (width 0.1) (type default)) (layer "F.SilkS"))
-    (fp_line (start 0 -0.75) (end 0 1.25)
-      (stroke (width 0.1) (type default)) (layer "F.SilkS"))
-    (fp_line (start 0 1.25) (end 0.25 1.5)
-      (stroke (width 0.1) (type default)) (layer "F.SilkS"))
-    (fp_line (start 0.25 1.5) (end 1 1.5)
-      (stroke (width 0.1) (type default)) (layer "F.SilkS"))
-    (fp_line (start 0.5 -1.25) (end 0 -0.75)
-      (stroke (width 0.1) (type default)) (layer "F.SilkS"))
-    (fp_line (start 1 1.5) (end 1.5 1)
-      (stroke (width 0.1) (type default)) (layer "F.SilkS"))
-    (fp_line (start 1.25 -1.25) (end 0.5 -1.25)
-      (stroke (width 0.1) (type default)) (layer "F.SilkS"))
-    (fp_line (start 1.5 -1) (end 1.25 -1.25)
-      (stroke (width 0.1) (type default)) (layer "F.SilkS"))
-    (fp_line (start 1.5 -0.5) (end 1.5 -1)
-      (stroke (width 0.1) (type default)) (layer "F.SilkS"))
-    (fp_line (start 1.5 0.25) (end 1 0.25)
-      (stroke (width 0.1) (type default)) (layer "F.SilkS"))
-    (fp_line (start 1.5 1) (end 1.5 0.25)
-      (stroke (width 0.1) (type default)) (layer "F.SilkS"))
-    (fp_circle (center 0 0) (end 0 -1.905)
+    (fp_line (start -1.016 -0.762) (end -0.508 0)
+      (stroke (width 0.1) (type default)) (layer "F.SilkS"))
+    (fp_line (start -0.508 0) (end -0.508 1.143)
+      (stroke (width 0.1) (type default)) (layer "F.SilkS"))
+    (fp_line (start -0.508 0) (end -0.127 -0.762)
+      (stroke (width 0.1) (type default)) (layer "F.SilkS"))
+    (fp_line (start 0 -0.508) (end 0 0.635)
+      (stroke (width 0.1) (type default)) (layer "F.SilkS"))
+    (fp_line (start 0 0.635) (end 0 0.889)
+      (stroke (width 0.1) (type default)) (layer "F.SilkS"))
+    (fp_line (start 0 0.889) (end 0.254 1.143)
+      (stroke (width 0.1) (type default)) (layer "F.SilkS"))
+    (fp_line (start 0.254 -0.762) (end 0 -0.508)
+      (stroke (width 0.1) (type default)) (layer "F.SilkS"))
+    (fp_line (start 0.254 1.143) (end 0.762 1.143)
+      (stroke (width 0.1) (type default)) (layer "F.SilkS"))
+    (fp_line (start 0.762 0.254) (end 0.508 0.254)
+      (stroke (width 0.1) (type default)) (layer "F.SilkS"))
+    (fp_line (start 0.762 1.143) (end 1.016 0.889)
+      (stroke (width 0.1) (type default)) (layer "F.SilkS"))
+    (fp_line (start 1.016 -0.762) (end 0.254 -0.762)
+      (stroke (width 0.1) (type default)) (layer "F.SilkS"))
+    (fp_line (start 1.016 0.254) (end 0.762 0.254)
+      (stroke (width 0.1) (type default)) (layer "F.SilkS"))
+    (fp_line (start 1.016 0.889) (end 1.016 0.254)
+      (stroke (width 0.1) (type default)) (layer "F.SilkS"))
+    (fp_circle (center 0 0) (end 0 -1.524)
       (stroke (width 0.1) (type default)) (fill none) (layer "F.SilkS"))
   )
@@
     (property "ki_keywords" "cap capacitor")
     (attr smd)
-    (fp_text reference "C3" (at 5.842 -2.413 90 unlocked) (layer "F.SilkS")
+    (fp_text reference "C3" (at 3.556 -2.032 90 unlocked) (layer "F.SilkS")
         (effects (font (size 1 1) (thickness 0.1)))
     )
@@
   )
   (footprint "Library:CapacitorSpecial" (layer "F.Cu")
-    (at 110.363 133.35 90)
+    (at 110.363 132.842 90)
     (property "Sheetfile" "snescart.kicad_sch")
     (property "Sheetname" "")
@@
   (gr_line (start 97.79 123.19) (end 93.98 123.19)
     (stroke (width 0.1) (type default)) (layer "Edge.Cuts"))
-  (gr_circle (center 100.33 118.11) (end 99.187 118.12051)
+  (gr_circle (center 100.33 118.11) (end 100.33 119.38)
     (stroke (width 0.1) (type default)) (fill none) (layer "Edge.Cuts"))
   (gr_line (start 115.57 151.13) (end 115.57 149.225)
@@
     (effects (font (size 1.5 1.5) (thickness 0.3) bold) (justify left bottom))
   )
-  (gr_text "MASK ROM" (at 179.959 115.697) (layer "F.SilkS")
-    (effects (font (size 1.5 1.5) (thickness 0.3) bold) (justify left bottom))
+  (gr_text "MASK ROM" (at 183.007 115.316) (layer "F.SilkS")
+    (effects (font (size 1 1) (thickness 0.2) bold) (justify left bottom))
   )
   (gr_text "1990" (at 98.679 135.255 90) (layer "F.SilkS")
     (effects (font (size 1.5 1.5) (thickness 0.3) bold) (justify left bottom))
   )
-  (segment (start 172.975 146.733) (end 172.975 139.318) (width 1.27) (layer "F.Cu") (net 1))
   (segment (start 180.34 137.795) (end 187.325 137.795) (width 1.905) (layer "F.Cu") (net 1))
   (segment (start 176.53 137.795) (end 178.435 137.795) (width 1.905) (layer "F.Cu") (net 1))
   (segment (start 178.435 137.795) (end 180.34 137.795) (width 1.905) (layer "F.Cu") (net 1))
+  (segment (start 172.975 140.334) (end 176.022 137.287) (width 1.27) (layer "F.Cu") (net 1))
   (segment (start 189.23 137.795) (end 193.04 137.795) (width 1.905) (layer "F.Cu") (net 1))
+  (segment (start 172.975 146.733) (end 172.975 140.334) (width 1.27) (layer "F.Cu") (net 1))
   (segment (start 193.04 137.795) (end 193.04 126.365) (width 1.905) (layer "F.Cu") (net 1))
-  (segment (start 172.975 139.318) (end 173.355 138.938) (width 1.27) (layer "F.Cu") (net 1))
   (segment (start 187.325 137.795) (end 189.23 137.795) (width 1.905) (layer "F.Cu") (net 1))
   (via (at 189.357 137.287) (size 0.8) (drill 0.4) (layers "F.Cu" "B.Cu") (net 1))
@@
   (via (at 179.07 137.287) (size 0.8) (drill 0.4) (layers "F.Cu" "B.Cu") (net 1))
   (via (at 186.817 137.287) (size 0.8) (drill 0.4) (layers "F.Cu" "B.Cu") (net 1))
-  (segment (start 138.049 133.223) (end 139.954 131.318) (width 1.905) (layer "F.Cu") (net 2))
+  (segment (start 114.808 131.953) (end 126.873 131.953) (width 1.905) (layer "F.Cu") (net 2))
   (segment (start 117.856 136.906) (end 117.856 134.62) (width 1.905) (layer "F.Cu") (net 2))
   (segment (start 128.27 133.223) (end 138.049 133.223) (width 1.905) (layer "F.Cu") (net 2))
   (segment (start 117.035 146.685) (end 117.035 139.895) (width 1.905) (layer "F.Cu") (net 2))
+  (segment (start 114.808 131.953) (end 114.808 137.033) (width 1.905) (layer "F.Cu") (net 2))
+  (segment (start 114.808 131.953) (end 117.729 131.953) (width 1.905) (layer "F.Cu") (net 2))
   (segment (start 117.856 134.62) (end 117.856 132.207) (width 1.905) (layer "F.Cu") (net 2))
   (segment (start 117.856 132.207) (end 117.856 132.08) (width 1.905) (layer "F.Cu") (net 2))
-  (segment (start 139.954 131.318) (end 139.954 123.063) (width 1.905) (layer "F.Cu") (net 2))
   (segment (start 117.035 139.895) (end 117.035 137.727) (width 1.905) (layer "F.Cu") (net 2))
+  (segment (start 126.873 131.953) (end 127.762 131.064) (width 1.905) (layer "F.Cu") (net 2))
+  (segment (start 117.729 134.62) (end 114.808 134.62) (width 1.905) (layer "F.Cu") (net 2))
+  (segment (start 114.808 137.033) (end 117.729 137.033) (width 1.905) (layer "F.Cu") (net 2))
   (segment (start 117.035 137.727) (end 117.856 136.906) (width 1.905) (layer "F.Cu") (net 2))
   (segment (start 117.729 134.62) (end 126.873 134.62) (width 1.905) (layer "F.Cu") (net 2))
   (segment (start 126.873 134.62) (end 128.27 133.223) (width 1.905) (layer "F.Cu") (net 2))
+  (via (at 114.808 131.953) (size 0.8) (drill 0.4) (layers "F.Cu" "B.Cu") (net 2))
   (via (at 117.729 137.033) (size 0.8) (drill 0.4) (layers "F.Cu" "B.Cu") (net 2))
   (via (at 117.729 134.62) (size 0.8) (drill 0.4) (layers "F.Cu" "B.Cu") (net 2))
   (via (at 117.729 131.953) (size 0.8) (drill 0.4) (layers "F.Cu" "B.Cu") (net 2))
+  (via (at 114.808 134.62) (size 0.8) (drill 0.4) (layers "F.Cu" "B.Cu") (net 2))
+  (via (at 114.808 137.033) (size 0.8) (drill 0.4) (layers "F.Cu" "B.Cu") (net 2))
   (segment (start 169.975 146.685) (end 169.975 143.256) (width 1.27) (layer "F.Cu") (net 37))
   (segment (start 174.244 130.175) (end 175.387 131.318) (width 0.25) (layer "F.Cu") (net 37))
