File: snescart.kicad_pcb (KiCad board)
At the start: 2 copper layers, 101.6 x 37.3 mm, 7 parts, among them P1 CASSETTE, U1 27C080

Commit message: back was messed up
Routing:
- net Net-(P1-A18): track 4.84 -> 12.6 mm
- net unconnected-(P1-A21-Pad46): track 7.22 -> 14.1 mm
- net unconnected-(P1-ROMSEL-Pad49): track 13.7 -> 19.1 mm
- net unconnected-(P1-A22-Pad47): track 16.5 -> 21.0 mm
- net unconnected-(P1-A20-Pad45): track 6.31 -> 9.91 mm
- net Net-(P1-D4): track 23.0 -> 26.3 mm
Changed lines of the file:
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@@
     (fp_line (start -1.016 -0.762) (end -0.508 0)
       (stroke (width 0.1) (type default)) (layer "F.SilkS"))
-    (fp_line (start -0.508 0) (end -0.508 1.016)
+    (fp_line (start -0.508 0) (end -0.508 0.762)
       (stroke (width 0.1) (type default)) (layer "F.SilkS"))
     (fp_line (start -0.508 0) (end -0.127 -0.762)
       (stroke (width 0.1) (type default)) (layer "F.SilkS"))
-    (fp_line (start 0 -0.508) (end 0 0.635)
-      (stroke (width 0.1) (type default)) (layer "F.SilkS"))
-    (fp_line (start 0 0.635) (end 0.254 1.016)
+    (fp_line (start 0 -0.508) (end 0 0.508)
+      (stroke (width 0.1) (type default)) (layer "F.SilkS"))
+    (fp_line (start 0 0.508) (end 0.254 0.762)
       (stroke (width 0.1) (type default)) (layer "F.SilkS"))
     (fp_line (start 0.254 -0.762) (end 0 -0.508)
       (stroke (width 0.1) (type default)) (layer "F.SilkS"))
-    (fp_line (start 0.254 1.016) (end 0.762 1.016)
+    (fp_line (start 0.254 0.762) (end 0.762 0.762)
       (stroke (width 0.1) (type default)) (layer "F.SilkS"))
     (fp_line (start 0.762 -0.762) (end 0.254 -0.762)
       (stroke (width 0.1) (type default)) (layer "F.SilkS"))
-    (fp_line (start 0.762 1.016) (end 1.016 0.762)
-      (stroke (width 0.1) (type default)) (layer "F.SilkS"))
-    (fp_line (start 1.016 0.1905) (end 0.508 0.1905)
-      (stroke (width 0.1) (type default)) (layer "F.SilkS"))
-    (fp_line (start 1.016 0.8255) (end 1.016 0.1905)
+    (fp_line (start 0.762 -0.762) (end 1.016 -0.508)
+      (stroke (width 0.1) (type default)) (layer "F.SilkS"))
+    (fp_line (start 0.762 0.762) (end 1.016 0.5715)
+      (stroke (width 0.1) (type default)) (layer "F.SilkS"))
+    (fp_line (start 1.016 0) (end 0.762 0)
+      (stroke (width 0.1) (type default)) (layer "F.SilkS"))
+    (fp_line (start 1.016 0.5715) (end 1.016 0)
       (stroke (width 0.1) (type default)) (layer "F.SilkS"))
     (fp_circle (center 0 0) (end 0 -1.524)
@@
   (segment (start 157.398 139.909) (end 160.147 137.16) (width 0.25) (layer "F.Cu") (net 40))
   (segment (start 154.811 140.718) (end 154.813 140.716) (width 0.25) (layer "F.Cu") (net 41))
+  (segment (start 154.811 139.956) (end 156.337 138.43) (width 0.25) (layer "F.Cu") (net 41))
+  (segment (start 154.811 145.559) (end 154.811 139.956) (width 0.25) (layer "F.Cu") (net 41))
   (segment (start 154.811 145.559) (end 154.811 140.718) (width 0.25) (layer "F.Cu") (net 41))
   (segment (start 152.351 145.559) (end 152.351 140.765) (width 0.25) (layer "F.Cu") (net 42))
@@
   (segment (start 184.15 118.618) (end 182.753 120.015) (width 0.254) (layer "B.Cu") (net 42))
   (segment (start 182.753 120.015) (end 181.61 120.015) (width 0.254) (layer "B.Cu") (net 42))
+  (segment (start 148.139181 132.715) (end 148.971 132.715) (width 0.254) (layer "F.Cu") (net 43))
   (segment (start 139.7762 139.8778) (end 141.224 138.43) (width 0.254) (layer "F.Cu") (net 43))
   (segment (start 145.034 136.144) (end 145.542 136.144) (width 0.254) (layer "F.Cu") (net 43))
@@
   (segment (start 141.224 138.43) (end 142.748 138.43) (width 0.254) (layer "F.Cu") (net 43))
   (segment (start 142.748 138.43) (end 145.034 136.144) (width 0.254) (layer "F.Cu") (net 43))
-  (segment (start 137.287 138.557) (end 137.287 146.304) (width 0.25) (layer "F.Cu") (net 44))
-  (segment (start 142.494 137.922) (end 137.922 137.922) (width 0.25) (layer "F.Cu") (net 44))
-  (segment (start 144.78 134.366) (end 144.78 135.636) (width 0.25) (layer "F.Cu") (net 44))
-  (segment (start 146.812 132.588) (end 148.59 130.81) (width 0.25) (layer "F.Cu") (net 44))
-  (segment (start 144.78 135.636) (end 142.494 137.922) (width 0.25) (layer "F.Cu") (net 44))
-  (segment (start 137.922 137.922) (end 137.287 138.557) (width 0.25) (layer "F.Cu") (net 44))
+  (segment (start 145.542 136.144) (end 147.463 134.223) (width 0.254) (layer "F.Cu") (net 43))
+  (segment (start 147.463 134.223) (end 147.463 133.391181) (width 0.254) (layer "F.Cu") (net 43))
+  (segment (start 147.463 133.391181) (end 148.139181 132.715) (width 0.254) (layer "F.Cu") (net 43))
+  (segment (start 145.792509 132.5245) (end 146.8755 132.5245) (width 0.25) (layer "F.Cu") (net 44))
+  (segment (start 137.287 138.557) (end 137.922 137.922) (width 0.25) (layer "F.Cu") (net 44))
+  (segment (start 144.78 133.537009) (end 145.792509 132.5245) (width 0.25) (layer "F.Cu") (net 44))
+  (segment (start 142.494 137.922) (end 144.78 135.636) (width 0.25) (layer "F.Cu") (net 44))
+  (segment (start 137.287 146.304) (end 137.287 138.557) (width 0.25) (layer "F.Cu") (net 44))
+  (segment (start 137.922 137.922) (end 142.494 137.922) (width 0.25) (layer "F.Cu") (net 44))
+  (segment (start 144.78 135.636) (end 144.78 133.537009) (width 0.25) (layer "F.Cu") (net 44))
+  (segment (start 146.8755 132.5245) (end 148.59 130.81) (width 0.25) (layer "F.Cu") (net 44))
   (via (at 148.59 130.81) (size 0.8) (drill 0.4) (layers "F.Cu" "B.Cu") (net 44))
   (segment (start 148.59 130.81) (end 148.59 133.604) (width 0.254) (layer "B.Cu") (net 44))
@@
   (segment (start 131.953 139.319) (end 133.223 138.049) (width 0.254) (layer "F.Cu") (net 49))
   (segment (start 149.891 145.559) (end 149.891 139.923) (width 0.25) (layer "F.Cu") (net 52))
+  (segment (start 151.384 138.43) (end 153.543 138.43) (width 0.25) (layer "F.Cu") (net 52))
+  (segment (start 150.368 139.446) (end 151.384 138.43) (width 0.25) (layer "F.Cu") (net 52))
   (segment (start 149.891 139.923) (end 150.368 139.446) (width 0.25) (layer "F.Cu") (net 52))
-  (segment (start 147.304 139.843) (end 148.336 138.811) (width 0.25) (layer "F.Cu") (net 53))
+  (segment (start 147.304 139.462) (end 148.844 137.922) (width 0.25) (layer "F.Cu") (net 53))
+  (segment (start 147.304 145.607) (end 147.304 139.462) (width 0.25) (layer "F.Cu") (net 53))
   (segment (start 147.304 145.607) (end 147.304 139.843) (width 0.25) (layer "F.Cu") (net 53))
+  (segment (start 146.558 137.16) (end 151.257 137.16) (width 0.25) (layer "F.Cu") (net 54))
+  (segment (start 151.257 137.16) (end 151.892 136.525) (width 0.25) (layer "F.Cu") (net 54))
   (segment (start 144.844 145.559) (end 144.844 138.874) (width 0.25) (layer "F.Cu") (net 54))
-  (segment (start 144.844 138.874) (end 147.32 136.398) (width 0.25) (layer "F.Cu") (net 54))
+  (segment (start 144.844 138.874) (end 146.558 137.16) (width 0.25) (layer "F.Cu") (net 54))
   (segment (start 144.844 145.559) (end 144.844 139.255) (width 0.25) (layer "F.Cu") (net 54))
   (segment (start 142.384 140.191) (end 143.764 138.811) (width 0.25) (layer "F.Cu") (net 55))
@@
         (xy 166.116 121.666)
         (xy 163.068 124.714)
-        (xy 163.068 125.984)
-        (xy 159.512 125.984)
-        (xy 157.48 123.952)
+        (xy 163.068 125.73)
+        (xy 162.687 126.111)
+        (xy 159.258 126.111)
+        (xy 157.226 123.952)
         (xy 152.908 123.952)
         (xy 151.384 125.222)

Commit message: ftghjdrftgh
Routing:
- net Net-(P1-A7): track 0.00 -> 81.4 mm
- net Net-(P1-A6): track 0.00 -> 69.6 mm
- net Net-(P1-A5): track 0.00 -> 65.9 mm
- net Net-(P1-A4): track 0.00 -> 62.6 mm
- net Net-(P1-A3): track 0.00 -> 59.1 mm
- net Net-(P1-A2): track 0.00 -> 55.5 mm
- net Net-(P1-A1): track 0.00 -> 51.7 mm
- net unconnected-(P1-A21-Pad46): track 14.1 -> 65.0 mm, vias 0 -> 1
- net Net-(P1-A0): track 0.00 -> 48.3 mm
- net unconnected-(P1-A22-Pad47): track 21.0 -> 63.7 mm, vias 0 -> 1
- net Net-(P1-D0): track 0.00 -> 42.7 mm
- net Net-(P1-A19): track 7.91 -> 45.8 mm
- net Net-(P1-A18): track 12.6 -> 48.4 mm, vias 0 -> 1
- net Net-(P1-A8): track 0.00 -> 31.9 mm
- net unconnected-(P1-RD-Pad23): track 10.4 -> 40.7 mm, vias 1 -> 2
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
Commit message: sdgs
Other:
- board text added: "C"
- board text added: "MASK"
- board text added: "N"
- board text added: "ROM"
- board text added: "n"
- board text added: "o"
- board text removed: "MASK ROM"

Commit message: backss
Routing:
- net unconnected-(P1-ROMSEL-Pad49): track 33.2 -> 62.9 mm
- net Net-(P1-A17): track 22.5 -> 48.0 mm
- net unconnected-(U2-NC-Pad10): track 0.00 -> 19.3 mm
- net Net-(P1-CIC3): track 35.2 -> 44.6 mm
- net Net-(P1-A19): track 45.8 -> 54.9 mm
- net unconnected-(U2-NC-Pad5): track 0.00 -> 6.82 mm
- net Net-(P1-A13): track 33.1 -> 39.7 mm, vias 0 -> 1
- net unconnected-(U2-NC-Pad3): track 0.00 -> 6.00 mm
- net Net-(P1-CIC2): track 45.7 -> 51.0 mm
- net unconnected-(U2-NC-Pad9): track 14.5 -> 18.4 mm
- net unconnected-(P1-RD-Pad23): track 40.7 -> 39.7 mm
- net Net-(P1-CIC1): track 20.3 -> 19.5 mm
- net unconnected-(P1-A20-Pad45): vias 1 -> 0
- net VCC: vias 11 -> 16
Other:
- outline, holes or cut-outs redrawn
